File: vdm2/vdm2.kicad_pcb (KiCad board)
At the start: 2 copper layers, 254 x 138.2 mm, 177 parts, among them IC1 7406, IC10 74LS109, IC11 74LS138, IC12 74LS86, IC13 74LS109, IC14 74LS02, IC15 74LS00, IC16 74LS109, IC17 74LS175, IC18 74LS132, IC19 74LS04, IC2 74LS163, IC20 74LS163, IC21 74LS163, IC22 74LS163, IC23 74LS157, IC24 74LS157, IC25 4049, IC26 4029, IC27 4029, IC28 74LS157, IC29 DM8131, IC3 74166, IC30 4001, IC31 4042, IC32 4042, IC33 74LS08, IC34 74LS08, IC35 74LS00, IC36 74LS04, IC37 8836, IC38 74LS367, IC39 74LS367, IC4 MCM6575, IC40 74LS10, IC41 2102, IC42 2102, IC43 2102, IC44 2102, IC45 2102, IC46 2102, IC47 2102, IC48 2102, IC49 L7805, IC5 74LS175, IC50 L7812, IC6 74LS175, IC7 74LS20, IC8 93L16, IC9 74LS10, J2 Jumper_3_Open, J4 Jumper_2_Open, J5 Jumper_2_Open, Q1 2N2907, SW1 SW_DIP_x06, Y1 Crystal

Commit message: Could it be a final version?
Parts:
- moved J2 38.4 mm to (195.2, 122.0), turned to 0 degrees
- moved R48 4.07 mm to (251.5, 140.3), turned to 180 degrees
- moved S100 4.06 mm to (55.4, 152.0)
Routing:
- net GND: track 2716.8 -> 2508.3 mm, vias 150 -> 142
- net Net-(IC31-Pad4): track 182.5 -> 366.2 mm, vias 4 -> 6
- net Net-(IC32-Pad7): track 305.5 -> 259.3 mm
- net Net-(IC36-Pad4): track 87.4 -> 126.6 mm, vias 1 -> 3
- net Net-(C39-Pad1): track 187.0 -> 162.6 mm, vias 3 -> 1
- net Net-(J2-Pad3): track 175.0 -> 151.1 mm, vias 1 -> 2
- net Net-(IC23-Pad6): track 123.9 -> 144.3 mm
- net Net-(IC28-Pad13): track 188.2 -> 171.9 mm
- net Net-(J2-Pad1): track 111.4 -> 95.8 mm, vias 0 -> 1
- net Net-(IC32-Pad14): track 229.3 -> 215.0 mm
- net Net-(C30-Pad2): track 169.2 -> 154.9 mm
- net Net-(IC29-Pad3): track 89.7 -> 76.4 mm
- net Net-(IC31-Pad13): track 180.9 -> 194.1 mm
- net Net-(IC34-Pad13): track 68.6 -> 55.9 mm
- net Net-(IC29-Pad5): track 88.1 -> 75.7 mm, vias 4 -> 3
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Other:
- board size 254 x 138.2 mm -> 254 x 134.1 mm
- board text added: "A10"
- board text added: "A11"
- board text added: "A12"
- board text added: "A13"
- board text added: "A14"
- board text added: "A15"
