File: kicad/vdm2021.kicad_pcb (KiCad board)
At the start: 2 copper layers, 254 x 134.1 mm, 177 parts, among them IC1 7406, IC10 74LS109, IC11 74LS138, IC12 74LS86, IC13 74LS109, IC14 74LS02, IC15 74LS00, IC16 74LS109, IC17 74LS175, IC18 74LS132, IC19 74LS04, IC2 74LS163, IC20 74LS163, IC21 74LS163, IC22 74LS163, IC23 74LS157, IC24 74LS157, IC25 4049, IC26 4029, IC27 4029, IC28 74LS157, IC29 DM8131, IC3 74166, IC30 4001, IC31 4042, IC32 4042, IC33 74LS08, IC34 74LS08, IC35 74LS00, IC36 74LS04, IC37 8836, IC38 74LS367, IC39 74LS367, IC4 MCM6575, IC40 74LS10, IC41 2102, IC42 2102, IC43 2102, IC44 2102, IC45 2102, IC46 2102, IC47 2102, IC48 2102, IC49 L7805, IC5 74LS175, IC50 L7812, IC6 74LS175, IC7 74LS20, IC8 93L16, IC9 74LS10, J2 Jumper_3_Open, J4 Jumper_2_Open, J5 Jumper_2_Open, Q1 2N2907, SW1 SW_DIP_x06, Y1 Crystal

Commit message: Moved video closer to top-edge.  Moved VDM-2021 silkscreen to left edge
Parts:
- removed VIDEO1: Conn_Coaxial, vdm2021:bnc-5-16345033
- added VIDEO: Conn_Coaxial, vdm2021:bnc-5-16345033, F.Cu at (262.3, 26.7)
Routing:
- net Net-(C1-Pad2): track 13.1 -> 21.6 mm
Changed lines of the file:
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@@
     (thickness 1.6)
     (drawings 22)
-    (tracks 5076)
+    (tracks 5077)
     (zones 0)
     (modules 177)
@@
   (page A3)
   (layers
-    (0 F.Cu signal hide)
+    (0 F.Cu signal)
     (31 B.Cu signal hide)
     (32 B.Adhes user hide)
@@
     (42 Eco1.User user hide)
     (43 Eco2.User user hide)
-    (44 Edge.Cuts user hide)
+    (44 Edge.Cuts user)
     (45 Margin user hide)
     (46 B.CrtYd user hide)
@@
   )
   (module vdm2021:bnc-5-16345033 locked (layer F.Cu)
-    (at 261.62 34.925 270)
+    (at 262.255 26.67 270)
     (descr 5-1634503-3-1)
     (tags Connector)
-    (fp_text reference VIDEO1 (at 0 0 270) (layer F.SilkS)
+    (fp_text reference VIDEO (at 6.223 0) (layer F.SilkS)
       (effects (font (size 1.27 1.27) (thickness 0.254)))
     )
@@
     )
   )
-  (gr_text "(rev 1)" (at 263.1186 25.2984) (layer F.Cu)
+  (gr_text "(rev 1)" (at 26.3652 25.527 90) (layer F.SilkS)
     (effects (font (size 1.016 1.016) (thickness 0.127)))
   )
@@
     (effects (font (size 2.032 2.032) (thickness 0.254)))
   )
-  (gr_text VDM-2021 (at 257.4798 21.6662) (layer F.SilkS)
+  (gr_text VDM-2021 (at 22.733 31.1658 90) (layer F.SilkS)
     (effects (font (size 3.81 2.54) (thickness 0.381)))
   )
@@
   (segment (start 102.374601 115.938399) (end 108.615689 115.938399) (width 0.2032) (layer B.Cu) (net 7))
   (segment (start 108.615689 115.938399) (end 111.257291 118.580001) (width 0.2032) (layer B.Cu) (net 7))
-  (segment (start 261.62 44.45) (end 261.62 34.925) (width 0.25) (layer F.Cu) (net 8))
+  (segment (start 261.62 27.305) (end 262.255 26.67) (width 0.25) (layer F.Cu) (net 8))
+  (segment (start 261.62 44.45) (end 261.62 27.305) (width 0.25) (layer F.Cu) (net 8))
   (segment (start 264.16 46.99) (end 261.62 44.45) (width 0.25) (layer F.Cu) (net 8))
   (segment (start 242.57 44.45) (end 245.999 44.45) (width 0.2032) (layer B.Cu) (net 9))
@@
       (pts
         (xy 271.145 144.907) (xy 264.795 144.907) (xy 264.795 41.529) (xy 259.715 41.529) (xy 254.635 41.529)
-        (xy 254.635 18.796) (xy 271.145 18.796)
+        (xy 254.635 18.415) (xy 271.145 18.415)
       )
     )
